File: kicad/voltmeter.kicad_pcb (KiCad board)
At the start: 2 copper layers, 167.6 x 66 mm, 62 parts, among them J1 Barrel_Jack, Q1 2N7000, Q2 2N7000, U1 MCP3428, U2 CD4060BM96, U3 MAX6951, U4 LM285Z-2.5

Commit message: schematic
Parts:
- added D7: ACSC02-41SURKWA-F01, footprints:ACSC02-41SURKWA-F01, F.Cu at (154.9, 60.9)
- added D8: LED, LED_SMD:LED_1206_3216Metric_Pad1.42x1.75mm_HandSolder, F.Cu at (163.6, 61.0)
- added Q3: 2N7000, Package_TO_SOT_SMD:SOT-23_Handsoldering, F.Cu at (30.2, 48.8)
- added Q4: 2N7000, Package_TO_SOT_SMD:SOT-23_Handsoldering, F.Cu at (30.2, 53.3)
- added R10: 4K7, Resistor_SMD:R_1206_3216Metric_Pad1.30x1.75mm_HandSolder, F.Cu at (24.1, 48.2)
- added R11: 4K7, Resistor_SMD:R_1206_3216Metric_Pad1.30x1.75mm_HandSolder, F.Cu at (24.1, 51.5)
- added R12: 4K7, Resistor_SMD:R_1206_3216Metric_Pad1.30x1.75mm_HandSolder, F.Cu at (24.1, 54.7)
- added R13: 4K7, Resistor_SMD:R_1206_3216Metric_Pad1.30x1.75mm_HandSolder, F.Cu at (24.1, 58.0)
- added SW1: SW_Push, Button_Switch_SMD:SW_SPST_B3SL-1022P, F.Cu at (154.9, 73.7)
- added TP1: TestPoint, TestPoint:TestPoint_Loop_D2.60mm_Drill1.6mm_Beaded, F.Cu at (45.7, 58.4)
- added TP2: TestPoint, TestPoint:TestPoint_Loop_D2.60mm_Drill1.6mm_Beaded, F.Cu at (45.7, 85.1)
- added TP3: TestPoint, TestPoint:TestPoint_Loop_D2.60mm_Drill1.6mm_Beaded, F.Cu at (45.7, 90.2)
- added TP4: TestPoint, TestPoint:TestPoint_Loop_D2.60mm_Drill1.6mm_Beaded, F.Cu at (45.7, 95.2)
- R9: value 680 -> 470
- moved U1 48.3 mm to (30.4, 73.7)
- moved U4 41.0 mm to (17.8, 86.4)
- moved R9 39.4 mm to (17.8, 94.0)
Connections:
- A1 pad 15: unconnected-(A1-Pad15) -> Net-(A1-2)
- U1 pad 7: SDA -> /i2c-levelshift/SDA_HV
- U1 pad 8: SCL -> /i2c-levelshift/SCL_LV
Routing:
- net (no net): track 98.5 -> 22.0 mm
- net Net-(D1-A): track 70.8 -> 0.00 mm, vias 1 -> 0
- net +5V: track 227.8 -> 284.1 mm, vias 5 -> 6
- net +2V5: track 188.1 -> 140.6 mm
- net Net-(A1-2): track 0.00 -> 25.0 mm
- net /difference-amplifier4/V_OUT: track 16.9 -> 0.00 mm
- net /difference-amplifier1/V_OUT: track 16.9 -> 0.00 mm
- net /difference-amplifier2/V_OUT: track 16.0 -> 0.00 mm
- net SCL: track 64.7 -> 61.6 mm
- net /difference-amplifier3/V_OUT: track 2.60 -> 0.00 mm
- net unconnected-(A1-RX-Pad19): track 0.63 -> 0.00 mm
- net unconnected-(A1-0-Pad16): track 0.63 -> 0.00 mm
- net unconnected-(A1-VBat-Pad9): track 0.63 -> 0.00 mm

Commit message: passes drc
Parts:
- removed the C6 at (196.8, 51.8)
- removed the C6 at (119.4, 81.3)
- removed the R1 at (177.8, 78.7)
- added C6: 100n, Capacitor_SMD:C_1206_3216Metric_Pad1.33x1.80mm_HandSolder, F.Cu at (193.0, 71.4)
- moved R12 112.9 mm to (134.6, 77.5), turned to 90 degrees
- moved R10 111.9 mm to (132.1, 77.5), turned to 90 degrees
- moved R11 82.6 mm to (101.6, 80.0), turned to 90 degrees
- moved R13 75.7 mm to (96.5, 80.0), turned to 90 degrees
- moved Q3 71.3 mm to (99.1, 67.3), turned to -90 degrees
- moved Q4 62.8 mm to (91.4, 67.3), turned to -90 degrees
- moved U4 58.0 mm to (74.9, 76.2), turned to -90 degrees
- moved U1 57.3 mm to (87.6, 77.5), turned to 90 degrees
- moved R9 54.6 mm to (69.8, 77.5)
Connections:
- Q4 pad 2: /i2c-levelshift/SCL_LV -> SCL
- Q4 pad 3: SCL -> /i2c-levelshift/SCL_HV
- R12 pad 2: /i2c-levelshift/SCL_LV -> SCL
- R13 pad 2: SCL -> /i2c-levelshift/SCL_HV
- U1 pad 8: /i2c-levelshift/SCL_LV -> /i2c-levelshift/SCL_HV
Routing:
- net +3V3: track 56.9 -> 256.9 mm, vias 0 -> 5
- net /difference-amplifier4/V_OUT: track 0.00 -> 105.1 mm, vias 0 -> 2
- net +2V5: track 140.6 -> 226.8 mm
- net Net-(A1-15): track 0.00 -> 85.9 mm, vias 0 -> 1
- net +5V: track 284.1 -> 357.4 mm, vias 6 -> 7
- net /difference-amplifier3/V_OUT: track 0.00 -> 67.6 mm, vias 0 -> 2
- net Net-(Q2-G): track 10.8 -> 68.8 mm
- net SCK: track 34.7 -> 86.1 mm
- net DISPLAY_CS: track 44.1 -> 93.9 mm
- net MOSI: track 39.5 -> 85.7 mm
- net GND: track 50.7 -> 9.05 mm
- net /difference-amplifier2/V_OUT: track 0.00 -> 38.5 mm
- net Net-(D1-A): track 0.00 -> 30.8 mm
- net /display/SEG1: track 61.6 -> 89.7 mm, vias 5 -> 6
- net SDA: track 22.6 -> 47.4 mm
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