File: kicad/7seg.kicad_sch (KiCad schematic)
At the start: 8 parts, among them U3 MAX6951

Commit message: schematic
Parts:
- added D7: ACSC02-41SURKWA-F01, footprints:ACSC02-41SURKWA-F01, symbol ACSC02-41SURKWA-F01:ACSC02-41SURKWA-F01
- added D8: LED, LED_SMD:LED_1206_3216Metric_Pad1.42x1.75mm_HandSolder, symbol Device:LED
Connections:
- net SEG0: now also D7.5 (DP), D8.2 (A)
- net SEG1: now also D7.10 (g)
- net SEG2: now also D7.9 (f)
- net SEG3: now also D7.1 (e)
- net SEG4: now also D7.3 (C.K.), D7.8 (C.K.)
- net SEG5: now also D7.2 (d), D8.1 (K)
- net SEG6: now also D7.4 (c)
- net SEG7: now also D7.6 (b)
- net SEG8: now also D7.7 (a)
Other:
- note added: "USED TO INDICATE NEGATIVE NUMBERS"
