File: kicad/voltmeter.kicad_sch (KiCad schematic)
At the start: 23 parts, among them J1 Barrel_Jack, Q1 2N7000, Q2 2N7000, U1 MCP3428, U2 CD4060BM96, U4 LM285Z-2.5

Commit message: schematic
Parts:
- added SW1: SW_Push, Button_Switch_SMD:SW_SPST_B3SL-1022P, symbol Switch:SW_Push
- added TP1, TP2, TP3, TP4: TestPoint, TestPoint:TestPoint_Loop_D2.60mm_Drill1.6mm_Beaded, symbol Connector:TestPoint
- R9: value 680 -> 470
Connections:
- net +2V5: now also TP4.1
- net +3V3: now also TP3.1
- net +5V: now also TP2.1
- net GND: now also SW1.1, TP1.1
- net SCL: no longer U1.8 (SCL)
- net SDA: no longer U1.7 (SDA)
- net at A1.15 (2): now also SW1.2
- new net i2c-levelshift/SCL_LV: U1.8 (SCL)
- new net i2c-levelshift/SDA_HV: U1.7 (SDA)
- no-connect marks 19 -> 18
Other:
- added sheet i2c-levelshift (i2c_levelshift.kicad_sch)
- note removed: "WIFI IS FUN"

Commit message: passes drc
Connections:
- net i2c-levelshift/SCL_LV renamed i2c-levelshift/SCL_HV
Changed lines of the file:
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@@
   (title_block
     (title "MQTT Voltmeter")
-    (date "2022-02-18")
-    (rev "A")
+    (date "2023-11-27")
+    (rev "B")
     (company "University of Wisconsin-Madison")
     (comment 1 "Department of Chemistry")
@@
       (effects (font (size 1.27 1.27)) (justify left top))
     )
-    (pin "SCL_LV" bidirectional (at 38.1 127 180)
-      (effects (font (size 1.27 1.27)) (justify left))
-    )
-    (pin "SCL_HV" bidirectional (at 63.5 127 0)
+    (pin "SCL_LV" bidirectional (at 63.5 127 0)
       (effects (font (size 1.27 1.27)) (justify right))
     )
+    (pin "SCL_HV" bidirectional (at 38.1 127 180)
+      (effects (font (size 1.27 1.27)) (justify left))
+    )
     (pin "SDA_HV" bidirectional (at 38.1 121.92 180)
